File: pots.sch (EAGLE design)
At the start: 6 parts

Commit message: Minor corrections
Connections:
- removed net VEE: JP2.1, JP2.3, JP2.5, JP2.7, JP2.9
- net VCC: now also JP2.1, JP2.3, JP2.5, JP2.7, JP2.9
Changed lines of the file:
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@@
 <part name="GND2" library="SparkFun" deviceset="GND" device=""/>
 <part name="GND3" library="SparkFun" deviceset="GND" device=""/>
-<part name="SUPPLY2" library="supply2" deviceset="VEE" device=""/>
 <part name="P+2" library="SparkFun" deviceset="VCC" device=""/>
 <part name="JP1" library="SparkFun" deviceset="M05X2" device="PTH"/>
@@
 <part name="GND1" library="SparkFun" deviceset="GND" device=""/>
 <part name="GND4" library="SparkFun" deviceset="GND" device=""/>
+<part name="P+4" library="SparkFun" deviceset="VCC" device=""/>
 </parts>
 <sheets>
@@
 <instance part="GND2" gate="1" x="106.68" y="121.92"/>
 <instance part="GND3" gate="1" x="137.16" y="152.4" rot="R180"/>
-<instance part="SUPPLY2" gate="G$1" x="137.16" y="121.92" rot="R180"/>
 <instance part="P+2" gate="1" x="106.68" y="149.86"/>
 <instance part="JP1" gate="G$1" x="106.68" y="137.16" rot="R90"/>
@@
 <instance part="GND1" gate="1" x="76.2" y="121.92"/>
 <instance part="GND4" gate="1" x="43.18" y="121.92"/>
+<instance part="P+4" gate="1" x="137.16" y="124.46" rot="R180"/>
 </instances>
 <busses>
@@
 <pinref part="P+3" gate="1" pin="VCC"/>
 </segment>
-</net>
-<net name="VEE" class="0">
 <segment>
 <wire x1="132.08" y1="129.54" x2="132.08" y2="127" width="0.1524" layer="91"/>
@@
 <junction x="134.62" y="127"/>
 <junction x="139.7" y="127"/>
-<pinref part="SUPPLY2" gate="G$1" pin="VEE"/>
 <pinref part="JP2" gate="G$1" pin="7"/>
 <pinref part="JP2" gate="G$1" pin="5"/>
@@
 <pinref part="JP2" gate="G$1" pin="1"/>
 <pinref part="JP2" gate="G$1" pin="9"/>
+<pinref part="P+4" gate="1" pin="VCC"/>
 </segment>
 </net>
