File: stereo-jack.sch (EAGLE design)
At the start: 4 parts, among them J1 STEREOSW

Commit message: Minor corrections
Connections:
- removed net VEE: JP2.1, JP2.3, JP2.5, JP2.7, JP2.9
- net N$1: no longer J1.SN
- net N$2: now also J1.R, JP3.3; no longer J1.T, J1.TN
- net N$3: now also J1.T, JP3.5; no longer J1.R, J1.RN, JP3.3
- net VCC: now also JP2.1, JP2.3, JP2.5, JP2.7, JP2.9; no longer JP3.5
Changed lines of the file:
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@@
 <part name="GND2" library="SparkFun" deviceset="GND" device=""/>
 <part name="GND3" library="SparkFun" deviceset="GND" device=""/>
-<part name="SUPPLY2" library="supply2" deviceset="VEE" device=""/>
 <part name="P+2" library="SparkFun" deviceset="VCC" device=""/>
 <part name="JP1" library="SparkFun" deviceset="M05X2" device="PTH"/>
 <part name="JP2" library="SparkFun" deviceset="M05X2" device="PTH"/>
 <part name="JP3" library="SparkFun" deviceset="M05" device="PTH"/>
-<part name="P+1" library="SparkFun" deviceset="VCC" device=""/>
 <part name="GND4" library="SparkFun" deviceset="GND" device=""/>
 <part name="J1" library="gm-jacks" deviceset="STEREOSW" device=""/>
+<part name="P+3" library="SparkFun" deviceset="VCC" device=""/>
 </parts>
 <sheets>
@@
 <instance part="GND2" gate="1" x="106.68" y="121.92"/>
 <instance part="GND3" gate="1" x="137.16" y="152.4" rot="R180"/>
-<instance part="SUPPLY2" gate="G$1" x="137.16" y="121.92" rot="R180"/>
 <instance part="P+2" gate="1" x="106.68" y="149.86"/>
 <instance part="JP1" gate="G$1" x="106.68" y="137.16" rot="R90"/>
 <instance part="JP2" gate="G$1" x="137.16" y="137.16" rot="R90"/>
 <instance part="JP3" gate="G$1" x="33.02" y="134.62"/>
-<instance part="P+1" gate="1" x="43.18" y="144.78"/>
 <instance part="GND4" gate="1" x="43.18" y="121.92"/>
 <instance part="J1" gate="G$1" x="71.12" y="134.62" rot="R180"/>
+<instance part="P+3" gate="1" x="137.16" y="124.46" rot="R180"/>
 </instances>
 <busses>
@@
 </segment>
 <segment>
-<wire x1="40.64" y1="139.7" x2="43.18" y2="139.7" width="0.1524" layer="91"/>
-<wire x1="43.18" y1="139.7" x2="43.18" y2="144.78" width="0.1524" layer="91"/>
-<pinref part="JP3" gate="G$1" pin="5"/>
-<pinref part="P+1" gate="1" pin="VCC"/>
-</segment>
-</net>
-<net name="VEE" class="0">
-<segment>
 <wire x1="132.08" y1="129.54" x2="132.08" y2="127" width="0.1524" layer="91"/>
 <wire x1="132.08" y1="127" x2="134.62" y2="127" width="0.1524" layer="91"/>
@@
 <junction x="134.62" y="127"/>
 <junction x="139.7" y="127"/>
-<pinref part="SUPPLY2" gate="G$1" pin="VEE"/>
 <pinref part="JP2" gate="G$1" pin="7"/>
 <pinref part="JP2" gate="G$1" pin="5"/>
@@
 <pinref part="JP2" gate="G$1" pin="1"/>
 <pinref part="JP2" gate="G$1" pin="9"/>
-</segment>
-</net>
-<net name="N$2" class="0">
-<segment>
-<pinref part="JP3" gate="G$1" pin="4"/>
-<wire x1="40.64" y1="137.16" x2="55.88" y2="137.16" width="0.1524" layer="91"/>
-<wire x1="55.88" y1="137.16" x2="55.88" y2="139.7" width="0.1524" layer="91"/>
-<pinref part="J1" gate="G$1" pin="T"/>
-<wire x1="55.88" y1="139.7" x2="58.42" y2="139.7" width="0.1524" layer="91"/>
-<pinref part="J1" gate="G$1" pin="TN"/>
-<wire x1="58.42" y1="139.7" x2="58.42" y2="142.24" width="0.1524" layer="91"/>
-</segment>
-</net>
-<net name="N$3" class="0">
-<segment>
-<pinref part="JP3" gate="G$1" pin="3"/>
-<pinref part="J1" gate="G$1" pin="R"/>
-<wire x1="40.64" y1="134.62" x2="58.42" y2="134.62" width="0.1524" layer="91"/>
-<pinref part="J1" gate="G$1" pin="RN"/>
-<wire x1="58.42" y1="134.62" x2="58.42" y2="137.16" width="0.1524" layer="91"/>
+<pinref part="P+3" gate="1" pin="VCC"/>
 </segment>
 </net>
@@
 <segment>
 <pinref part="JP3" gate="G$1" pin="2"/>
-<pinref part="J1" gate="G$1" pin="SN"/>
+<wire x1="40.64" y1="132.08" x2="53.34" y2="132.08" width="0.1524" layer="91"/>
+<wire x1="53.34" y1="132.08" x2="53.34" y2="129.54" width="0.1524" layer="91"/>
 <pinref part="J1" gate="G$1" pin="S"/>
-<wire x1="40.64" y1="132.08" x2="58.42" y2="132.08" width="0.1524" layer="91"/>
-<wire x1="58.42" y1="132.08" x2="58.42" y2="129.54" width="0.1524" layer="91"/>
+<wire x1="53.34" y1="129.54" x2="58.42" y2="129.54" width="0.1524" layer="91"/>
 </segment>
 </net>
+<net name="N$2" class="0">
+<segment>
+<pinref part="JP3" gate="G$1" pin="3"/>
+<pinref part="J1" gate="G$1" pin="R"/>
+<wire x1="40.64" y1="134.62" x2="48.26" y2="134.62" width="0.1524" layer="91"/>
+<pinref part="JP3" gate="G$1" pin="4"/>
+<wire x1="48.26" y1="134.62" x2="58.42" y2="134.62" width="0.1524" layer="91"/>
+<wire x1="40.64" y1="137.16" x2="48.26" y2="137.16" width="0.1524" layer="91"/>
+<wire x1="48.26" y1="137.16" x2="48.26" y2="134.62" width="0.1524" layer="91"/>
+</segment>
+</net>
+<net name="N$3" class="0">
+<segment>
+<pinref part="JP3" gate="G$1" pin="5"/>
+<pinref part="J1" gate="G$1" pin="T"/>
+<wire x1="40.64" y1="139.7" x2="58.42" y2="139.7" width="0.1524" layer="91"/>
+</segment>
+</net>
